File: KiCad/Ouroboros/DaisySeed.kicad_sch (KiCad schematic)
At the start: 0 parts

Commit message: Updating schematic
Parts:
- added A1: Electrosmith_Daisy_Seed_Rev4, Module:Electrosmith_Daisy_Seed, symbol MCU_Module:Electrosmith_Daisy_Seed_Rev4
- added C10: 1u, symbol Device:C
- added C9: 100n, symbol Device:C
- added RV2, RV3, RV4, RV5, RV6, RV7: B10k, symbol Device:R_Potentiometer
- added SW2, SW3, SW4: SW_Push, symbol Switch:SW_Push
Connections:
- new net +3V3: A1.21 (3V3_A), RV2.1, RV3.1, RV4.1, RV5.1, RV6.1, RV7.1
- new net +9V: A1.39 (VIN), C10.1, C9.1
- new net Blend_Knob: A1.26 (ADC_4), RV6.2
- new net FDBK_Knob: A1.23 (ADC_1), RV3.2
- new net Filt_Knob: A1.27 (ADC_5), RV7.2
- new net GND: A1.17 (AUDIO_IN_2), A1.20 (AGND), A1.40 (DGND), C10.2, C9.2, RV2.3, RV3.3, RV4.3, RV5.3, RV6.3, RV7.3, SW2.2, SW3.2, SW4.2
- new net I2C_SCL: A1.12 (I2C1_SCL)
- new net I2C_SDA: A1.13 (I2C1_SDA)
- new net IN_GAIN: A1.16 (AUDIO_IN_1)
- new net OUT_L: A1.18 (AUDIO_OUT_1)
- new net OUT_R: A1.19 (AUDIO_OUT_2)
- new net Rate_Knob: A1.22 (ADC_0), RV2.2
- new net SW_1: A1.32 (SAI2_SD_B), SW2.1
- new net SW_2: A1.33 (SAI2_SD_A), SW3.1
- new net SW_3: A1.34 (SAI2_FS), SW4.1
- new net Space_Knob: A1.24 (ADC_2), RV4.2
- new net Wow_Knob: A1.25 (ADC_3), RV5.2
Other:
- note added: "Knobs"
- note added: "Seed"
- note added: "Switches"
- note added: "[1] Daisy Seed"

Commit message: Linking nets
Changed lines of the file:
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@@
+		)
+	)
+	(hierarchical_label "OUT_L"
+		(shape input)
+		(at 96.52 77.47 180)
+		(fields_autoplaced yes)
+		(effects
+			(font
+				(size 1.27 1.27)
+			)
+			(justify right)
+		)
+	)
+	(hierarchical_label "I2C_SDA"
+		(shape input)
+		(at 191.77 90.17 0)
+		(fields_autoplaced yes)
+		(effects
+			(font
+				(size 1.27 1.27)
+			)
+			(justify left)
+		)
+	)
+	(hierarchical_label "OUT_R"
+		(shape input)
+		(at 96.52 80.01 180)
+		(fields_autoplaced yes)
+		(effects
+			(font
+				(size 1.27 1.27)
+			)
+			(justify right)
+		)
+	)
+	(hierarchical_label "I2C_SCL"
+		(shape input)
+		(at 191.77 87.63 0)
+		(fields_autoplaced yes)
+		(effects
+			(font
+				(size 1.27 1.27)
+			)
+			(justify left)
+		)
+	)
+	(hierarchical_label "IN_GAIN"
+		(shape input)
+		(at 96.52 72.39 180)
+		(fields_autoplaced yes)
+		(effects
+			(font
+				(size 1.27 1.27)
+			)
+			(justify right)
 		)
 	)

Commit message: Updated schematic, started PCB
Parts:
- C10: footprint (none) -> Capacitor_THT:C_Rect_L7.0mm_W6.0mm_P5.00mm
- C9: footprint (none) -> Capacitor_THT:C_Rect_L7.0mm_W3.5mm_P5.00mm
- RV2, RV3, RV4, RV5, RV6, RV7: footprint (none) -> Potentiometer_THT:Potentiometer_Alpha_RD901F-40-00D_Single_Vertical
- SW2, SW3, SW4: footprint (none) -> Button_Switch_Keyboard:SW_Cherry_MX_1.00u_PCB
Changed lines of the file:
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@@
 			)
 		)
-		(property "Footprint" ""
+		(property "Footprint" "Capacitor_THT:C_Rect_L7.0mm_W6.0mm_P5.00mm"
 			(at 124.1552 52.07 0)
 			(effects
@@
 			)
 		)
-		(property "Footprint" ""
+		(property "Footprint" "Potentiometer_THT:Potentiometer_Alpha_RD901F-40-00D_Single_Vertical"
 			(at 36.83 140.97 0)
 			(effects
@@
 			)
 		)
-		(property "Footprint" ""
+		(property "Footprint" "Potentiometer_THT:Potentiometer_Alpha_RD901F-40-00D_Single_Vertical"
 			(at 36.83 170.18 0)
 			(effects
@@
 			)
 		)
-		(property "Footprint" ""
+		(property "Footprint" "Capacitor_THT:C_Rect_L7.0mm_W3.5mm_P5.00mm"
 			(at 135.5852 52.07 0)
 			(effects
@@
 			)
 		)
-		(property "Footprint" ""
+		(property "Footprint" "Potentiometer_THT:Potentiometer_Alpha_RD901F-40-00D_Single_Vertical"
 			(at 100.33 170.18 0)
 			(effects
@@
 			)
 		)
-		(property "Footprint" ""
+		(property "Footprint" "Button_Switch_Keyboard:SW_Cherry_MX_1.00u_PCB"
 			(at 245.11 113.03 0)
 			(effects
@@
 			)
 		)
-		(property "Footprint" ""
+		(property "Footprint" "Potentiometer_THT:Potentiometer_Alpha_RD901F-40-00D_Single_Vertical"
 			(at 128.27 170.18 0)
 			(effects
@@
 			)
 		)
-		(property "Footprint" ""
+		(property "Footprint" "Potentiometer_THT:Potentiometer_Alpha_RD901F-40-00D_Single_Vertical"
 			(at 158.75 170.18 0)
 			(effects
@@
 			)
 		)
-		(property "Footprint" ""
+		(property "Footprint" "Button_Switch_Keyboard:SW_Cherry_MX_1.00u_PCB"
 			(at 245.11 138.43 0)
 			(effects
@@
 			)
 		)
-		(property "Footprint" ""
+		(property "Footprint" "Button_Switch_Keyboard:SW_Cherry_MX_1.00u_PCB"
 			(at 245.11 125.73 0)
 			(effects
@@
 			)
 		)
-		(property "Footprint" ""
+		(property "Footprint" "Potentiometer_THT:Potentiometer_Alpha_RD901F-40-00D_Single_Vertical"
 			(at 69.85 170.18 0)
 			(effects

Commit message: PCB Finished
Parts:
- added D4, D5, D6, D7, D8, D9: LED, LED_THT:LED_D3.0mm, symbol Device:LED
- added R17, R18, R19, R20, R21, R22: 1k, Resistor_THT:R_Axial_DIN0207_L6.3mm_D2.5mm_P10.16mm_Horizontal, symbol Device:R
Connections:
- net GND: now also D4.1 (K), D5.1 (K), D6.1 (K), D7.1 (K), D8.1 (K), D9.1 (K)
- net LED_4: now reaches A1.2 (SD_DATA_3)
- net LED_4: now also R22.2
- net LED_3: now reaches A1.3 (SD_DATA_2)
- net LED_3: now also R21.2
- net LED_2: now reaches A1.4 (SD_DATA_1)
- net LED_2: now also R17.2
- net LED_1: now reaches A1.5 (SD_DATA_0)
- net LED_1: now also R18.2
- net LED_5: now reaches A1.6 (SD_CMD)
- net LED_5: now also R20.2
- net LED_6: now reaches A1.7 (SD_CLK)
- net LED_6: now also R19.2
- new net: D4.2 (A), R17.1
- new net: D5.2 (A), R18.1
- new net: D6.2 (A), R19.1
- new net: D8.2 (A), R21.1
- new net: D9.2 (A), R22.1
- new net: D7.2 (A), R20.1
Other:
- note added: "LEDs"

Commit message: Dev Board complete
Parts:
- added SW5: SW_Push, Button_Switch_Keyboard:SW_Cherry_MX_1.00u_PCB, symbol Switch:SW_Push
Connections:
- net GND: now also SW5.2; no longer A1.17 (AUDIO_IN_2)
- net SEND_SW: now reaches A1.11 (SPI1_PICO)
- net SW_4: now reaches A1.31 (SAI2_MCLK)
- net SW_4: now also SW5.1
- new net IN_L: A1.17 (AUDIO_IN_2)
