File: KiCad/Ouroboros/Ouroboros.kicad_pcb (KiCad board)
At the start: 4 copper layers, 165.1 x 127 mm, 48 parts, among them J1 AudioJack2, J2 Jack-DC, J3 AudioJack2, J4 AudioJack2, SW1 SW_DPDT_x2, SW2 SW_Push, SW3 SW_Push, SW4 SW_Push, U1 Opamp_Quad, U3 LM78L05_TO92

Commit message: PCB Finished
Parts:
- added C17: 1u, Capacitor_THT:C_Rect_L7.0mm_W6.0mm_P5.00mm, F.Cu at (308.6, 174.0)
- added C18: 1u, Capacitor_THT:C_Rect_L7.0mm_W6.0mm_P5.00mm, F.Cu at (308.6, 182.9)
- added C19: 1u, Capacitor_THT:C_Rect_L7.0mm_W6.0mm_P5.00mm, F.Cu at (313.6, 165.1)
- added C20: 1u, Capacitor_THT:C_Rect_L7.0mm_W6.0mm_P5.00mm, F.Cu at (313.6, 156.2)
- added D4: LED, LED_THT:LED_D3.0mm, F.Cu at (289.5, 208.0)
- added D5: LED, LED_THT:LED_D3.0mm, F.Cu at (289.5, 200.0)
- added D6: LED, LED_THT:LED_D3.0mm, F.Cu at (289.2, 184.0)
- added D7: LED, LED_THT:LED_D3.0mm, F.Cu at (289.5, 192.0)
- added D8: LED, LED_THT:LED_D3.0mm, F.Cu at (289.5, 216.0)
- added D9: LED, LED_THT:LED_D3.0mm, F.Cu at (289.5, 224.0)
- added H1: GND, TestPoint:TestPoint_THTPad_D1.5mm_Drill0.7mm, F.Cu at (420.0, 155.0)
- added H2: VCC, TestPoint:TestPoint_THTPad_D1.5mm_Drill0.7mm, F.Cu at (422.5, 155.0)
- added H3: SCL, TestPoint:TestPoint_THTPad_D1.5mm_Drill0.7mm, F.Cu at (425.0, 155.0)
- added H4: SDA, TestPoint:TestPoint_THTPad_D1.5mm_Drill0.7mm, F.Cu at (427.5, 155.0)
- added R12: 470k, Resistor_THT:R_Axial_DIN0207_L6.3mm_D2.5mm_P10.16mm_Horizontal, F.Cu at (321.3, 185.4)
- added R13: 100R, Resistor_THT:R_Axial_DIN0207_L6.3mm_D2.5mm_P10.16mm_Horizontal, F.Cu at (327.7, 157.5)
- added R14: 100R, Resistor_THT:R_Axial_DIN0207_L6.3mm_D2.5mm_P10.16mm_Horizontal, F.Cu at (331.5, 167.6)
- added R15: 100k, Resistor_THT:R_Axial_DIN0207_L6.3mm_D2.5mm_P10.16mm_Horizontal, F.Cu at (318.8, 149.9)
- added R16: 100k, Resistor_THT:R_Axial_DIN0207_L6.3mm_D2.5mm_P10.16mm_Horizontal, F.Cu at (290.8, 149.9)
- added R17: 1k, Resistor_THT:R_Axial_DIN0207_L6.3mm_D2.5mm_P10.16mm_Horizontal, F.Cu at (323.9, 199.0)
- added R18: 1k, Resistor_THT:R_Axial_DIN0207_L6.3mm_D2.5mm_P10.16mm_Horizontal, F.Cu at (307.0, 199.0)
- added R19: 1k, Resistor_THT:R_Axial_DIN0207_L6.3mm_D2.5mm_P10.16mm_Horizontal, F.Cu at (306.8, 191.0)
- added R20: 1k, Resistor_THT:R_Axial_DIN0207_L6.3mm_D2.5mm_P10.16mm_Horizontal, F.Cu at (306.9, 195.0)
- added R21: 1k, Resistor_THT:R_Axial_DIN0207_L6.3mm_D2.5mm_P10.16mm_Horizontal, F.Cu at (323.8, 203.2)
- added R22: 1k, Resistor_THT:R_Axial_DIN0207_L6.3mm_D2.5mm_P10.16mm_Horizontal, F.Cu at (323.8, 207.2)
- added R9: 470k, Resistor_THT:R_Axial_DIN0207_L6.3mm_D2.5mm_P10.16mm_Horizontal, F.Cu at (326.4, 180.3)
- C16: value 100p -> 1u; footprint Capacitor_THT:C_Rect_L7.0mm_W3.5mm_P5.00mm -> Capacitor_THT:C_Rect_L7.0mm_W6.0mm_P5.00mm
- moved A1 158.8 mm to (447.7, 193.0), turned to -90 degrees
- moved C9 158.6 mm to (447.0, 212.5), turned to -90 degrees
- moved C10 146.0 mm to (441.0, 212.5), turned to -90 degrees
- moved RV2 84.4 mm to (297.8, 244.0), turned to 90 degrees
- moved RV7 61.9 mm to (368.0, 226.7), turned to 90 degrees
- moved U1 60.3 mm to (355.6, 176.5), turned to 180 degrees
- moved RV3 49.4 mm to (312.6, 226.7), turned to 90 degrees
- moved RV6 46.5 mm to (354.9, 244.0), turned to 90 degrees
- moved C8 46.0 mm to (362.0, 169.0), turned to 0 degrees
- moved C16 44.5 mm to (396.3, 156.2)
- moved D2 43.7 mm to (396.2, 161.3)
- moved D1 43.6 mm to (391.2, 168.9)
- moved R8 43.6 mm to (401.3, 171.4)
- moved C15 39.7 mm to (387.4, 161.3), turned to -90 degrees
- moved RV4 36.2 mm to (327.1, 244.0), turned to 90 degrees
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Connections:
- net /InputOutput/IN_BUF renamed /Input/IN_BUF
- net /InputOutput/Inst_Level renamed /Input/Inst_Level
- net /InputOutput/Line_Level renamed /Input/Line_Level
- A1 pad 2: unconnected-(A1-SD_DATA_3-Pad2) -> /DaisySeed/LED_4
- A1 pad 3: unconnected-(A1-SD_DATA_2-Pad3) -> /DaisySeed/LED_3
- A1 pad 4: unconnected-(A1-SD_DATA_1-Pad4) -> /DaisySeed/LED_2
- A1 pad 5: unconnected-(A1-SD_DATA_0-Pad5) -> /DaisySeed/LED_1
- A1 pad 6: unconnected-(A1-SD_CMD-Pad6) -> /DaisySeed/LED_5
- A1 pad 7: unconnected-(A1-SD_CLK-Pad7) -> /DaisySeed/LED_6
- J1 pad SN: (no net) -> GND
- J1 pad TN: (no net) -> GND
- J2 pad MP: (no net) -> GND
- J3 pad SN: (no net) -> GND
- J3 pad T: Net-(J3-PadT) -> Net-(C19-Pad2)
- J3 pad TN: (no net) -> GND
- J4 pad SN: (no net) -> GND
- J4 pad T: Net-(J4-PadT) -> Net-(C20-Pad2)
- J4 pad TN: (no net) -> GND
- RV8 pad 2: Net-(J4-PadT) -> Net-(C18-Pad1)
- RV8 pad 5: Net-(J3-PadT) -> Net-(C17-Pad1)
- U1 pad 10: (no net) -> Net-(U1C-+)
- U1 pad 12: (no net) -> Net-(U1D-+)
- U1 pad 13: (no net) -> Net-(U1D--)
- U1 pad 14: (no net) -> Net-(U1D--)
- U1 pad 8: (no net) -> Net-(U1C--)
- U1 pad 9: (no net) -> Net-(U1C--)
Routing:
- net +3V3: track 0.00 -> 157.8 mm
- net /DaisySeed/Rate_Knob: track 0.00 -> 132.9 mm
- net /DaisySeed/LED_1: track 0.00 -> 131.9 mm, vias 0 -> 1
- net /OUT_L: track 0.00 -> 130.8 mm
- net /OUT_R: track 0.00 -> 129.5 mm
- net /DaisySeed/LED_5: track 0.00 -> 125.3 mm, vias 0 -> 1
- net /DaisySeed/LED_6: track 0.00 -> 122.7 mm, vias 0 -> 1
- net /DaisySeed/LED_4: track 0.00 -> 119.2 mm
- net +5V: track 0.00 -> 119.1 mm
- net /DaisySeed/LED_3: track 0.00 -> 117.4 mm
- net /DaisySeed/LED_2: track 0.00 -> 116.0 mm
- net /DaisySeed/Space_Knob: track 0.00 -> 109.2 mm
- net /DaisySeed/FDBK_Knob: track 0.00 -> 102.0 mm
- net /DaisySeed/Blend_Knob: track 0.00 -> 85.8 mm
- net /DaisySeed/Wow_Knob: track 0.00 -> 77.9 mm
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- added copper zone on B.Cu, net +2V5
- added copper zone on B.Cu, net +5V
- added copper zone on B.Cu, net +9V
- added copper zone on B.Cu, net GND
- added copper zone on F.Cu, net GND
- added copper zone on In1.Cu, net GND
- added copper zone on In2.Cu, net GND
- added copper zone on B.Cu, net Net-(D3-A)
Other:
- board text added: "1"
- board text added: "12/06/2024"
- board text added: "15"
- board text added: "16"
- board text added: "17"
- board text added: "18"
- board text added: "19"
- board text added: "2"
- board text added: "20"
- board text added: "25"
- board text added: "26"
- board text added: "27"
- board text added: "3"
- board text added: "4"
- board text added: "5"
- board text added: "6"
- board text added: "Blend"
- board text added: "Div"
- board text added: "Eaz Audio"
- board text added: "FDBK"
- board text added: "Filter"
- board text added: "Ouroboros Dev V1"
- board text added: "Preset"
- board text added: "Rate"
- board text added: "Space"
- board text added: "Tap"
- board text added: "Wow"

Commit message: Dev Board complete
Parts:
- added C21: 100p, Capacitor_THT:C_Rect_L7.0mm_W3.5mm_P5.00mm, F.Cu at (424.2, 166.8)
- added C22: 1u, Capacitor_THT:C_Rect_L7.0mm_W6.0mm_P5.00mm, F.Cu at (418.5, 166.8)
- added C23: 1n, Capacitor_THT:C_Rect_L7.0mm_W3.5mm_P5.00mm, F.Cu at (431.0, 177.2)
- added C24: 100n, Capacitor_THT:C_Rect_L7.0mm_W3.5mm_P5.00mm, F.Cu at (415.5, 187.8)
- added J5: AudioJack2, Connector_Audio:Jack_6.35mm_Neutrik_NMJ4HFD2_Horizontal, F.Cu at (396.4, 139.0)
- added Q1: BF244A, Package_TO_SOT_THT:TO-92_Inline, F.Cu at (288.6, 171.2)
- added R23: 1k, Resistor_THT:R_Axial_DIN0207_L6.3mm_D2.5mm_P10.16mm_Horizontal, F.Cu at (428.1, 175.8)
- added R24: 470k, Resistor_THT:R_Axial_DIN0207_L6.3mm_D2.5mm_P10.16mm_Horizontal, F.Cu at (441.1, 181.8)
- added R25: 0R, Resistor_THT:R_Axial_DIN0204_L3.6mm_D1.6mm_P1.90mm_Vertical, F.Cu at (406.9, 184.8)
- added R26: 0R, Resistor_THT:R_Axial_DIN0204_L3.6mm_D1.6mm_P1.90mm_Vertical, F.Cu at (406.6, 189.5)
- added R27: 0R, Resistor_THT:R_Axial_DIN0204_L3.6mm_D1.6mm_P1.90mm_Vertical, F.Cu at (366.6, 173.8)
- added R28: 0R, Resistor_THT:R_Axial_DIN0204_L3.6mm_D1.6mm_P1.90mm_Vertical, F.Cu at (401.5, 174.0)
- added R29: 0R, Resistor_THT:R_Axial_DIN0204_L3.6mm_D1.6mm_P1.90mm_Vertical, F.Cu at (300.5, 172.7)
- added R30: 0R, Resistor_THT:R_Axial_DIN0204_L3.6mm_D1.6mm_P1.90mm_Vertical, F.Cu at (304.5, 172.7)
- added R31: 1k, Resistor_THT:R_Axial_DIN0207_L6.3mm_D2.5mm_P10.16mm_Horizontal, F.Cu at (294.5, 181.1)
- added R32: 1k, Resistor_THT:R_Axial_DIN0207_L6.3mm_D2.5mm_P10.16mm_Horizontal, F.Cu at (297.8, 170.9)
- added R33: 0R, Resistor_THT:R_Axial_DIN0207_L6.3mm_D2.5mm_P10.16mm_Horizontal, F.Cu at (393.4, 169.1)
- added R34: 0R, Resistor_THT:R_Axial_DIN0207_L6.3mm_D2.5mm_P10.16mm_Horizontal, F.Cu at (397.0, 169.1)
- added R35: 1k, Resistor_THT:R_Axial_DIN0207_L6.3mm_D2.5mm_P10.16mm_Horizontal, F.Cu at (353.8, 197.6)
- added SW5: SW_Push, Button_Switch_Keyboard:SW_Cherry_MX_1.00u_PCB, F.Cu at (381.4, 225.9)
- added U2: Opamp_Dual, Package_DIP:DIP-8_W7.62mm_Socket, F.Cu at (427.8, 187.6)
- moved C13 39.8 mm to (400.5, 186.8), turned to 180 degrees
- moved R8 35.0 mm to (392.0, 137.7), turned to -90 degrees
- moved C3 34.8 mm to (413.0, 168.0), turned to 180 degrees
- moved C2 26.2 mm to (422.7, 153.2)
- moved C1 26.2 mm to (422.7, 160.8)
- moved R1 26.2 mm to (412.6, 164.6)
- moved R3 26.2 mm to (407.5, 154.4)
- moved D1 19.2 mm to (403.3, 154.0), turned to 180 degrees
- moved D2 10.8 mm to (395.7, 150.5), turned to 0 degrees
- moved R5 10.2 mm to (384.0, 178.9), turned to -90 degrees
- moved H1 10.1 mm to (429.2, 151.0)
- moved H2 10.1 mm to (431.8, 151.0)
- moved H3 10.1 mm to (434.2, 151.0)
- moved H4 10.1 mm to (436.8, 151.0)
- moved RV7 7.55 mm to (360.5, 226.7)
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Connections:
- A1 pad 11: unconnected-(A1-SPI1_PICO-Pad11) -> /SEND_SW
- A1 pad 17: GND -> /DaisySeed/IN_L
- A1 pad 31: unconnected-(A1-SAI2_MCLK-Pad31) -> /DaisySeed/SW_4
- C16 pad 2: /DaisySeed/IN_GAIN -> Net-(C16-Pad2)
- C3 pad 1: Net-(U1A-+) -> Net-(U2B-+)
- R1 pad 1: Net-(U1A-+) -> Net-(U2B-+)
- R11 pad 2: /Gain/IN_LEVEL -> Net-(R11-Pad2)
- R3 pad 2: Net-(U1A-+) -> Net-(U2B-+)
- R6 pad 2: /Gain/IN_LEVEL -> Net-(R11-Pad2)
- R8 pad 2: /DaisySeed/IN_GAIN -> Net-(C16-Pad2)
- RV8 pad 1: GND -> Net-(Q1-D)
- RV8 pad 3: /OUT_R -> Net-(R30-Pad2)
- RV8 pad 6: /OUT_L -> Net-(R29-Pad2)
- U1 pad 1: /Input/IN_BUF -> (no net)
- U1 pad 2: /Input/IN_BUF -> (no net)
- U1 pad 3: Net-(U1A-+) -> (no net)
Routing:
- net /SEND_SW: track 0.00 -> 141.1 mm
- net +2V5: track 52.2 -> 184.5 mm
- net Net-(U1A-+): track 73.4 -> 0.00 mm
- net +5V: track 119.1 -> 185.6 mm
- net /DaisySeed/SW_4: track 0.00 -> 52.7 mm
- net Net-(C21-Pad1): track 0.00 -> 42.7 mm
- net Net-(C16-Pad2): track 0.00 -> 34.1 mm
- net Net-(U2B-+): track 0.00 -> 24.7 mm
- net Net-(U2A--): track 0.00 -> 24.5 mm
- net Net-(SW1B-B): track 37.7 -> 16.1 mm
- net /DaisySeed/IN_GAIN: track 41.4 -> 20.5 mm
- net /Gain/IN_LEVEL: track 32.2 -> 16.0 mm
- net Net-(U2B--): track 0.00 -> 15.9 mm
- net Net-(R11-Pad2): track 0.00 -> 15.7 mm
- net /OUT_R: track 129.5 -> 116.8 mm
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Other:
- board text added: "24"
- board text added: "Gain"
- board text added: "INST"
- board text added: "IN_BUF_L"
- board text added: "IN_BUF_R"
- board text added: "IN_GAIN"
- board text added: "IN_L"
- board text added: "IN_LEVEL_L"
- board text added: "IN_R RETURN"
- board text added: "LINE"
- board text added: "OUT_L"
- board text added: "OUT_R"
- board text added: "OUT_R SEND"
- board text added: "On/Off"
- board text added: "Vol"
