File: KiCad/Ouroboros/input.kicad_sch (KiCad schematic)
At the start: 14 parts, among them J1 AudioJack2, SW1 SW_DPDT_x2, U1 Opamp_Quad

Commit message: Dev Board complete
Parts:
- removed U1: Opamp_Quad, Package_DIP:DIP-14_W7.62mm_Socket, symbol Amplifier_Operational:TL074
- added C21: 100p, Capacitor_THT:C_Rect_L7.0mm_W3.5mm_P5.00mm, symbol Device:C
- added C22: 1u, Capacitor_THT:C_Rect_L7.0mm_W6.0mm_P5.00mm, symbol Device:C
- added C23: 1n, Capacitor_THT:C_Rect_L7.0mm_W3.5mm_P5.00mm, symbol Device:C
- added J5: AudioJack2, Connector_Audio:Jack_6.35mm_Neutrik_NMJ4HFD2_Horizontal, symbol Connector_Audio:NMJ4HFD2
- added R23: 1k, Resistor_THT:R_Axial_DIN0207_L6.3mm_D2.5mm_P10.16mm_Horizontal, symbol Device:R
- added R24: 470k, Resistor_THT:R_Axial_DIN0207_L6.3mm_D2.5mm_P10.16mm_Horizontal, symbol Device:R
- added R25, R26, R27: 0R, Resistor_THT:R_Axial_DIN0204_L3.6mm_D1.6mm_P1.90mm_Vertical, symbol Device:R
- added U2: Opamp_Dual, Package_DIP:DIP-8_W7.62mm_Socket, symbol Device:Opamp_Dual
Connections:
- net +2V5: now also R24.1
- net GND: now also C21.2, C23.2, J5.S, J5.SN, J5.TN
- net IN_BUF: now also R25.2
- net at C3.1, R1.1, R3.2: now also U2.5 (+)
- net IN_LEVEL: no longer names the net of R11.2, R6.2
- net IN_LEVEL: now also R27.1
- new net: R26.1, U2.1, U2.2 (-)
- new net: C23.1, R23.1, R24.2, U2.3 (+)
- new net: R25.1, U2.6 (-), U2.7
- new net: C21.1, C22.1, J5.T
- new net: C22.2, R23.2
- new net IN_BUF_R: R26.2
- new net IN_LEVEL_L: R27.2
Other:
- note added: "L Input Buffer"
- note added: "R Input Buffer"
- note removed: "Input Buffer"
- moved on the sheet: C12, C13, C3, R11, R4, R5, R6, SW1A, SW1B
